File: hardware/FLORADASH-PCB.kicad_sch (KiCad schematic)
At the start: 76 parts, among them IC1 LM66200DRLR, J1 USB_C_Receptacle_USB2.0_16P, J2 Conn_01x04_Pin, J3 Conn_02x04_Top_Bottom, Q1 FS8205, Q2 FS8205, SW1 SW_Push, SW2 SW_Push, U1 TP4056-42-ESOP8, U2 USBLC6-2SC6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

Commit message: Routing structure
Parts:
- L2: footprint Inductor_SMD:L_0603_1608Metric -> Inductor_SMD:L_1008_2520Metric; JLCPCB Part # (none) -> C354538
- TP1, TP2, TP3, TP4, TP5, TP6: footprint TestPoint:TestPoint_Pad_D2.5mm -> TestPoint:TestPoint_Pad_D1.0mm

Commit message: Placement of components on PCB
Parts:
- U6: footprint Connector_PinSocket_2.54mm:PinSocket_1x03_P2.54mm_Vertical -> Connector_PinSocket_2.54mm:PinSocket_1x03_P2.54mm_Horizontal
Changed lines of the file:
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@@
 			)
 		)
-		(property "Footprint" "Connector_PinSocket_2.54mm:PinSocket_1x03_P2.54mm_Vertical"
+		(property "Footprint" "Connector_PinSocket_2.54mm:PinSocket_1x03_P2.54mm_Horizontal"
 			(at 222.25 120.65 0)
 			(hide yes)

Commit message: signal routing
Parts:
- removed H2: MountingHole, MountingHole:MountingHole_2.2mm_M2_DIN965_Pad, symbol Mechanical:MountingHole
Changed lines of the file:
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@@
-	)
-	(symbol
-		(lib_id "Mechanical:MountingHole")
-		(at 196.85 157.48 0)
-		(unit 1)
-		(body_style 1)
-		(exclude_from_sim no)
-		(in_bom no)
-		(on_board yes)
-		(in_pos_files yes)
-		(dnp no)
-		(fields_autoplaced yes)
-		(property "Reference" "H2"
-			(at 199.39 157.4799 0)
-			(show_name no)
-			(do_not_autoplace no)
-			(effects
-				(font
-					(size 1.27 1.27)
-				)
-				(justify left)
-			)
-		)
-		(property "Value" "MountingHole"
-			(at 199.39 158.7499 0)
-			(hide yes)
-			(show_name no)
-			(do_not_autoplace no)
-			(effects
-				(font
-					(size 1.27 1.27)
-				)
-				(justify left)
-			)
-		)
-		(property "Footprint" "MountingHole:MountingHole_2.2mm_M2_DIN965_Pad"
-			(at 196.85 157.48 0)
-			(hide yes)
-			(show_name no)
-			(do_not_autoplace no)
-			(effects
-				(font
-					(size 1.27 1.27)
-				)
-			)
-		)
-		(property "Datasheet" ""
-			(at 196.85 157.48 0)
-			(hide yes)
-			(show_name no)
-			(do_not_autoplace no)
-			(effects
-				(font
-					(size 1.27 1.27)
-				)
-			)
-		)
-		(property "Description" "Mounting Hole without connection"
-			(at 196.85 157.48 0)
-			(hide yes)
-			(show_name no)
-			(do_not_autoplace no)
-			(effects
-				(font
-					(size 1.27 1.27)
-				)
-			)
-		)
-		(property "JLCPCB Part #" ""
-			(at 196.85 157.48 0)
-			(hide yes)
-			(show_name no)
-			(do_not_autoplace no)
-			(effects
-				(font
-					(size 1.27 1.27)
-				)
-			)
-		)
-		(property "Sim.Device" ""
-			(at 196.85 157.48 0)
-			(hide yes)
-			(show_name no)
-			(do_not_autoplace no)
-			(effects
-				(font
-					(size 1.27 1.27)
-				)
-			)
-		)
-		(property "Sim.Type" ""
-			(at 196.85 157.48 0)
-			(hide yes)
-			(show_name no)
-			(do_not_autoplace no)
-			(effects
-				(font
-					(size 1.27 1.27)
-				)
-			)
-		)
-		(property "PROD_ID" ""
-			(at 196.85 157.48 0)
-			(hide yes)
-			(show_name no)
-			(do_not_autoplace no)
-			(effects
-				(font
-					(size 1.27 1.27)
-				)
-			)
-		)
-		(property "Tolerance" ""
-			(at 196.85 157.48 0)
-			(hide yes)
-			(show_name no)
-			(do_not_autoplace no)
-			(effects
-				(font
-					(size 1.27 1.27)
-				)
-			)
-		)
-		(property "Voltage" ""
-			(at 196.85 157.48 0)
-			(hide yes)
-			(show_name no)
-			(do_not_autoplace no)
-			(effects
-				(font
-					(size 1.27 1.27)
-				)
-			)
-		)
-		(instances
-			(project "FLORADASH-PCB"
-				(path "/cead742e-00ff-4eab-9d80-942a293a1b5f"
-					(reference "H2")
-					(unit 1)
-				)
-			)
-		)
 	)
 	(symbol

Commit message: finish the first routing
Parts:
- renumbered H3 to H2, H4 to H3
Changed lines of the file:
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@@
 		(in_pos_files yes)
 		(dnp no)
-		(property "Reference" "H3"
+		(property "Reference" "H2"
 			(at 191.77 162.56 0)
 			(show_name no)
@@
 			(project "FLORADASH-PCB"
 				(path "/cead742e-00ff-4eab-9d80-942a293a1b5f"
-					(reference "H3")
+					(reference "H2")
 					(unit 1)
 				)
@@
 		(dnp no)
 		(fields_autoplaced yes)
-		(property "Reference" "H4"
+		(property "Reference" "H3"
 			(at 199.39 162.5599 0)
 			(show_name no)
@@
 			(project "FLORADASH-PCB"
 				(path "/cead742e-00ff-4eab-9d80-942a293a1b5f"
-					(reference "H4")
+					(reference "H3")
 					(unit 1)
 				)

Commit message: Finished the footprint assignation and PCB
Parts:
- BT1, H1, H2, H3: now not fitted
- DS1: JLCPCB Part # (none) -> C2718488; now in the parts list
- J2: JLCPCB Part # (none) -> C2718488
- J3: JLCPCB Part # (none) -> C225519
- R9: footprint Connector_PinSocket_2.00mm:PinSocket_1x02_P2.00mm_Vertical -> Connector_PinSocket_2.54mm:PinSocket_1x02_P2.54mm_Vertical; JLCPCB Part # (none) -> C49661
- SW1, SW2: JLCPCB Part # (none) -> C2886894
- TP1, TP2, TP3, TP4, TP5, TP6: now not fitted; now left out of the parts list
- U6: JLCPCB Part # (none) -> C22438144
- U7: JLCPCB Part # (none) -> C2759924
Changed lines of the file:
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@@
 		(body_style 1)
 		(exclude_from_sim no)
-		(in_bom yes)
+		(in_bom no)
 		(on_board yes)
 		(in_pos_files yes)
-		(dnp no)
+		(dnp yes)
 		(property "Reference" "TP5"
 			(at 276.098 23.368 0)
@@
 		(body_style 1)
 		(exclude_from_sim no)
-		(in_bom yes)
+		(in_bom no)
 		(on_board yes)
 		(in_pos_files yes)
-		(dnp no)
+		(dnp yes)
 		(property "Reference" "TP1"
 			(at 53.086 20.574 0)
@@
 		(body_style 1)
 		(exclude_from_sim no)
-		(in_bom yes)
+		(in_bom no)
 		(on_board yes)
 		(in_pos_files yes)
-		(dnp no)
+		(dnp yes)
 		(property "Reference" "TP6"
 			(at 107.696 81.534 0)
@@
 			)
 		)
+		(property "JLCPCB Part #" "C2886894"
+			(at 111.76 176.53 90)
+			(hide yes)
+			(show_name no)
+			(do_not_autoplace no)
+			(effects
+				(font
+					(size 1.27 1.27)
+				)
+			)
+		)
 		(pin "1"
 		)
@@
 			)
 		)
-		(property "JLCPCB Part #" ""
+		(property "JLCPCB Part #" "C22438144"
 			(at 222.25 120.65 0)
 			(hide yes)
@@
 			)
 		)
+		(property "JLCPCB Part #" "C2886894"
+			(at 86.36 179.07 90)
+			(hide yes)
+			(show_name no)
+			(do_not_autoplace no)
+			(effects
+				(font
+					(size 1.27 1.27)
+				)
+			)
+		)
 		(pin "1"
 		)
@@
 		(on_board yes)
 		(in_pos_files yes)
-		(dnp no)
+		(dnp yes)
 		(property "Reference" "H2"
 			(at 191.77 162.56 0)
@@
 		(body_style 1)
 		(exclude_from_sim no)
-		(in_bom yes)
+		(in_bom no)
 		(on_board yes)
 		(in_pos_files yes)
-		(dnp no)
+		(dnp yes)
 		(property "Reference" "TP3"
 			(at 192.786 21.844 0)
@@
 		(body_style 1)
 		(exclude_from_sim no)
-		(in_bom yes)
+		(in_bom no)
 		(on_board yes)
 		(in_pos_files yes)
-		(dnp no)
+		(dnp yes)
 		(property "Reference" "TP2"
 			(at 87.376 20.574 0)
@@
 			)
 		)
-		(property "JLCPCB Part #" ""
+		(property "JLCPCB Part #" "C2718488"
 			(at 146.05 171.45 0)
 			(hide yes)
@@
 		(body_style 1)
 		(exclude_from_sim no)
-		(in_bom yes)
+		(in_bom no)
 		(on_board yes)
 		(in_pos_files yes)
-		(dnp no)
+		(dnp yes)
 		(property "Reference" "TP4"
 			(at 256.54 23.114 0)
@@
 		(on_board yes)
 		(in_pos_files yes)
-		(dnp no)
+		(dnp yes)
 		(fields_autoplaced yes)
 		(property "Reference" "H3"
@@
 		(on_board yes)
 		(in_pos_files yes)
-		(dnp no)
+		(dnp yes)
 		(fields_autoplaced yes)
 		(property "Reference" "BT1"
@@
 		(body_style 1)
 		(exclude_from_sim no)
-		(in_bom no)
+		(in_bom yes)
 		(on_board yes)
 		(in_pos_files yes)
@@
 			)
 		)
-		(property "JLCPCB Part #" ""
+		(property "JLCPCB Part #" "C2718488"
 			(at 229.87 152.4 0)
 			(hide yes)
@@
 			)
 		)
+		(property "JLCPCB Part #" "C225519 "
+			(at 157.48 182.88 0)
+			(hide yes)
+			(show_name no)
+			(do_not_autoplace no)
+			(effects
+				(font
+					(size 1.27 1.27)
+				)
+			)
+		)
 		(pin "6"
 		)
@@
 			)
 		)
-		(property "Footprint" "Connector_PinSocket_2.00mm:PinSocket_1x02_P2.00mm_Vertical"
+		(property "Footprint" "Connector_PinSocket_2.54mm:PinSocket_1x02_P2.54mm_Vertical"
 			(at 256.54 76.2 90)
 			(hide yes)
@@
 			)
 		)
-		(property "JLCPCB Part #" ""
+		(property "JLCPCB Part #" "C49661"
 			(at 255.27 69.85 90)
 			(hide yes)
@@
 			)
 		)
+		(property "JLCPCB Part #" "C2759924"
+			(at 148.59 135.89 0)
+			(hide yes)
+			(show_name no)
+			(do_not_autoplace no)
+			(effects
+				(font
+					(size 1.27 1.27)
+				)
+			)
+		)
 		(pin "7"
 		)
@@
 		(on_board yes)
 		(in_pos_files yes)
-		(dnp no)
+		(dnp yes)
 		(fields_autoplaced yes)
 		(property "Reference" "H1"

Commit message: Finished routing PCB
Parts:
- removed U4: MT3420SP, Package_SO:SOIC-8_3.9x4.9mm_P1.27mm, symbol MT3420SP:MT3420SP
- added U4: (no value), SY8089BAAC:SY8089AAAC_SGY, symbol SY8089BAAC_SGY:SY8089BAAC
- C1, C13, C15, C17, C18, C19, C2, C4, C5, C9: JLCPCB Part # (none) -> C14663
- C10, C11, C12, C7, C8: JLCPCB Part # (none) -> C59461
- C14: JLCPCB Part # (none) -> C15849
- C16: JLCPCB Part # (none) -> C1604
- C3: JLCPCB Part # (none) -> C19702
- C6: JLCPCB Part # (none) -> C1653
- L1: value 2n2 -> 2u2; footprint Inductor_SMD:L_0603_1608Metric -> Inductor_SMD:L_1008_2520Metric; JLCPCB Part # (none) -> C354538
- R1, R10, R18, R4, R6, R8: JLCPCB Part # (none) -> C21190
- R11: JLCPCB Part # (none) -> C25804
- R12: JLCPCB Part # (none) -> C2998118
- R13: JLCPCB Part # (none) -> C177513
- R14: JLCPCB Part # (none) -> C23204
- R15, R17: JLCPCB Part # (none) -> C23182
- R16: JLCPCB Part # (none) -> C4190
- R19, R2, R3: JLCPCB Part # (none) -> C23186
- R20, R21: JLCPCB Part # (none) -> C23162
- R5: JLCPCB Part # (none) -> C22765
- R7: JLCPCB Part # (none) -> C22775
- SW1, SW2: JLCPCB Part # C2886894 -> C778172
- U6: now in the parts list
Connections:
- net GND: now also U4.2 (GND)
- net battery/usb: now also U4.1 (EN), U4.4 (IN)
- net at C6.2, R12.1, R13.2: now also U4.5 (FB)
- net at L2.1: now also U4.3 (LX)
